File: templates/Library.kicad_blocks/ldo 3.3v.kicad_block/ldo 3.3v.kicad_sch (KiCad schematic)
At the start: 3 parts, among them U1 SGM2212-3.3XKC3G/TR_C3294699

Commit message: update
Parts:
- U1: footprint kicad-libraries:SOT-223-3_L6.5-W3.4-P2.30-LS7.0-BR -> Z_IU3qez:SOT-223-3_L6.5-W3.4-P2.30-LS7.0-BR
Connections:
- net 3.3V renamed +3.3V
Other:
- moved on the sheet: C1, C2, U1
